File: UR3ILF_SI5351/KiCAD_PCB/UR3ILF.sch (KiCad schematic (older format))
At the start: 76 parts, among them J1 SPI, J2 ENCODER, J3 Conn_01x30, J4 CAT, J5 Conn_01x01, J6 Conn_01x01, J7 Conn_01x01, SW1 SW_Push, SW2 SW_Push, SW3 SW_Push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

Commit message: PCB almost ready
Connections:
- net CW: now reaches J3.5 (Pin_5), U6.6 (QG)
Changed lines of the file:
@@
 	4050 4900 4500 4900
 Wire Wire Line
-	4500 4900 4500 6700
+	4500 4900 4500 7350
 Wire Wire Line
 	4050 4800 4650 4800
 Wire Wire Line
-	4650 4800 4650 6700
+	4650 4800 4650 7200
 Wire Wire Line
 	4050 4400 5850 4400
@@
 	0    1    1    0
 $EndComp
-Text GLabel 4650 6700 3    60   Output ~ 0
+Text GLabel 5000 7200 2    60   Output ~ 0
 PREAMP
-Text GLabel 4500 6700 3    60   Output ~ 0
+Text GLabel 5000 7350 2    60   Output ~ 0
 ATT
-Text GLabel 2350 2000 0    60   Output ~ 0
+Text GLabel 2350 2000 0    60   Input ~ 0
 PTT
-Text GLabel 12100 2800 0    60   Input ~ 0
+Text GLabel 12100 2800 0    60   Output ~ 0
 PTT
 Text GLabel 12100 3500 0    60   Input ~ 0
@@
 P 10750 6100
 F 0 "J5" H 10750 6200 50  0000 C CNN
-F 1 "Conn_01x01" H 10750 6000 50  0000 C CNN
+F 1 "Conn_01x01" H 10750 6000 50  0001 C CNN
 F 2 "footprints:MountingHole_3.2mm_M3_DIN965_Pad" H 10750 6100 50  0001 C CNN
 F 3 "" H 10750 6100 50  0001 C CNN
@@
 P 10550 6100
 F 0 "#PWR47" H 10550 5850 50  0001 C CNN
-F 1 "GND" H 10550 5950 50  0000 C CNN
+F 1 "GND" H 10550 5950 50  0001 C CNN
 F 2 "" H 10550 6100 50  0001 C CNN
 F 3 "" H 10550 6100 50  0001 C CNN
@@
 P 10750 6500
 F 0 "J6" H 10750 6600 50  0000 C CNN
-F 1 "Conn_01x01" H 10750 6400 50  0000 C CNN
+F 1 "Conn_01x01" H 10750 6400 50  0001 C CNN
 F 2 "footprints:MountingHole_3.2mm_M3_DIN965_Pad" H 10750 6500 50  0001 C CNN
 F 3 "" H 10750 6500 50  0001 C CNN
@@
 P 10550 6500
 F 0 "#PWR53" H 10550 6250 50  0001 C CNN
-F 1 "GND" H 10550 6350 50  0000 C CNN
+F 1 "GND" H 10550 6350 50  0001 C CNN
 F 2 "" H 10550 6500 50  0001 C CNN
 F 3 "" H 10550 6500 50  0001 C CNN
@@
 P 10750 6950
 F 0 "J7" H 10750 7050 50  0000 C CNN
-F 1 "Conn_01x01" H 10750 6850 50  0000 C CNN
+F 1 "Conn_01x01" H 10750 6850 50  0001 C CNN
 F 2 "footprints:MountingHole_3.2mm_M3_DIN965_Pad" H 10750 6950 50  0001 C CNN
 F 3 "" H 10750 6950 50  0001 C CNN
@@
 P 10550 6950
 F 0 "#PWR56" H 10550 6700 50  0001 C CNN
-F 1 "GND" H 10550 6800 50  0000 C CNN
+F 1 "GND" H 10550 6800 50  0001 C CNN
 F 2 "" H 10550 6950 50  0001 C CNN
 F 3 "" H 10550 6950 50  0001 C CNN
@@
 	5250 4600 5250 6250
 Wire Wire Line
-	5150 6250 5150 4500
+	5150 4500 5150 6250
 Wire Wire Line
 	5150 4500 4050 4500
@@
 Text Label 12100 1900 0    60   ~ 0
 A3
+Wire Wire Line
+	4650 7200 5000 7200
+Wire Wire Line
+	4500 7350 5000 7350
+Text Label 12100 1600 0    60   ~ 0
+CW
 $EndSCHEMATC
