File: Raisin.kicad_pcb (KiCad board)
At the start: 2 copper layers, 95.5 x 100 mm, 224 parts, among them CON1 AVR_ISP, J1 CW_KEY, J10 Encoder, J11 i2c, J12 Barrel_Jack, J13 PA, J14 Conn_01x02, J15 TX, J2 Line OUT, J3 MIC, J4 ANT_PA, J5 Conn_01x01, J6 Conn_01x01, J7 Conn_01x01, J8 Conn_01x01, J9 PTT, Q1 MMBFJ310LT1G, Q10 BSS138, Q11 2N7002, Q2 MMBFJ310LT1G, Q3 Si2301-TP, Q4 Si2301-TP, Q5 2N7002, Q6 MMBT3906, Q7 MMBFJ310LT1G, Q8 2N7002, Q9 2N7002, T1 1:2, T2 Transformer, T3 Transformer, T4 Transformer, U1 ATMEGA328P-AU, U10 L78L06_TO92, U2 Si5351, U3 NE5532, U4 SA612A, U5 LD1117S33TR_SOT223, U6 L78L05_TO92, U7 FSA3157L6X, U8 TDA7052A, Y1 Crystal_GND23_Small, Y10 Crystal_GND23_Small, Y11 Crystal_GND23_Small, Y12 Crystal_GND23_Small, Y13 Crystal_GND23_Small, Y2 27Mhz, Y3 Crystal_GND23_Small, Y4 Crystal_GND23_Small, Y5 Crystal_GND23_Small, Y6 Crystal_GND23_Small, Y7 Crystal_GND23_Small, Y8 Crystal_GND23_Small, Y9 Crystal_GND23_Small

Commit message: PCB almost ready
Parts:
- removed C18, C31, C42, C55, C61, C89, C92, C93, C94: 100nF, Capacitors_SMD:C_0603_HandSoldering
- removed C3, C4, C7, C8: 22pF, raisin:C_1206_0603
- removed C32: 33uF, Capacitors_ThroughHole:CP_Radial_D6.3mm_P2.50mm
- removed C40, C50, C53, C56, C57, C59, C75: 10nF, Capacitors_SMD:C_0603_HandSoldering
- removed C43, C71, C90, C91: 1uF, raisin:C_1206_0603
- removed C51: 4n7, raisin:C_1206_0603
- removed C54: 47n, raisin:C_1206_0603
- removed C58, C62: 10uF, Capacitors_ThroughHole:CP_Radial_D4.0mm_P2.00mm
- removed C70: 270, raisin:C_1206_0603
- removed C78, C81: 100pF, raisin:C_1206_0603
- removed CON1: AVR_ISP, Pin_Headers:Pin_Header_Straight_2x03_Pitch2.54mm
- removed D14: BB132, Diodes_SMD:D_SOD-323_HandSoldering
- removed D8: LL4148, Diodes_SMD:D_MiniMELF
- removed L1: L_Small, raisin:Choke_Toroid_6,5x13mm_Vertical
- removed L10: 8.5uH, raisin:Choke_Toroid_6,5x13mm_Vertical
- removed L2, L5: 47uH, Resistors_ThroughHole:R_Axial_DIN0204_L3.6mm_D1.6mm_P7.62mm_Horizontal
- removed L7, L9: 22uH, Resistors_ThroughHole:R_Axial_DIN0204_L3.6mm_D1.6mm_P7.62mm_Horizontal
- removed LS1: Speaker, Buzzers_Beepers:BUZZER
- removed Q10: BSS138, TO_SOT_Packages_SMD:SOT-23
- removed Q6: MMBT3906, TO_SOT_Packages_SMD:SOT-23
- removed Q9: 2N7002, TO_SOT_Packages_SMD:SOT-23
- removed R1: 150k*, raisin:R_1206_0603
- removed R21, R31, R39: 1k, Resistors_SMD:R_0603_HandSoldering
- removed R27: 150, raisin:R_1206_0603
- removed R29, R37: 300k, raisin:R_1206_0603
- removed R30, R33, R34: 15k, raisin:R_1206_0603
- removed R35: 300*, raisin:R_1206_0603
- removed R4, R5: 4.7k, Resistors_SMD:R_0603_HandSoldering
- removed R40, R41: 470k, raisin:R_1206_0603
- removed R43, R6: 100, raisin:R_1206_0603
- removed R46: 10k, raisin:R_1206_0603
- removed RV1, RV3: POT, raisin:Potentiometer_WH148
- removed T3, T4: Transformer, raisin:TF14
- removed U10: L78L06_TO92, TO_SOT_Packages_THT:TO-92_Molded_Wide
- removed U4: SA612A, raisin:DIP-8_SOIC-8_W7.62mm
- removed U8: TDA7052A, Housings_DIP:DIP-8_W7.62mm
- removed Y1, Y3: Crystal_GND23_Small, raisin:Crystal_HC49-U_Vertical
- added C100: 100nF, Capacitors_SMD:C_0603_HandSoldering, B.Cu at (124.9, 141.7)
- added C101: 100nF, raisin:C_1206_0603, B.Cu at (116.4, 121.2)
- added C103: 10nF, Capacitors_SMD:C_0603_HandSoldering, B.Cu at (112.1, 127.4)
- added C104: 100nF, raisin:C_1206_0603, B.Cu at (124.1, 129.4)
- added C105: 10pF*, raisin:C_1206_0603, B.Cu at (106.8, 132.7)
- added C106: 10nF, Capacitors_SMD:C_0603_HandSoldering, B.Cu at (102.8, 122.1)
- added C107: 10nF, Capacitors_SMD:C_0603_HandSoldering, B.Cu at (101.1, 129.4)
- added C108: 100nF, raisin:C_1206_0603, B.Cu at (97.6, 134.4)
- added C109: 10nF, Capacitors_SMD:C_0603_HandSoldering, B.Cu at (126.4, 160.7)
- added C110: 10nF, Capacitors_SMD:C_0603_HandSoldering, B.Cu at (117.6, 158.1)
- added C111: 22pF*/100nF, raisin:C_1206_0603, B.Cu at (85.6, 122.7)
- added C112: 22pF, raisin:C_1206_0603, B.Cu at (88.0, 118.9)
- added C113: 100nF, raisin:C_1206_0603, B.Cu at (88.7, 125.8)
- added C114: 10uF, Capacitors_ThroughHole:CP_Radial_D4.0mm_P2.00mm, F.Cu at (89.7, 129.5)
- added C115: 10nF, Capacitors_SMD:C_0603_HandSoldering, B.Cu at (82.2, 121.7)
- added C116: 10nF, Capacitors_SMD:C_0603_HandSoldering, B.Cu at (83.8, 134.0)
- added C117: 10uF, Capacitors_ThroughHole:CP_Radial_D4.0mm_P2.00mm, F.Cu at (57.9, 128.8)
- added C118: 100nF, raisin:C_1206_0603, B.Cu at (57.0, 132.1)
- added C95: 100nF, raisin:C_1206_0603, B.Cu at (90.0, 56.1)
- added C96: 100nF, raisin:C_1206_0603, B.Cu at (124.2, 123.4)
- added C97: 100nF, raisin:C_1206_0603, B.Cu at (124.1, 126.7)
- added C98: 100pF, raisin:C_1206_0603, B.Cu at (120.5, 136.6)
- added C99: 180pF, raisin:C_1206_0603, B.Cu at (125.1, 139.2)
- added J16: MIC, raisin:audio_jack_3_5mm_PJ307, F.Cu at (113.5, 160.0)
- added J17: BPF, Pin_Headers:Pin_Header_Straight_1x02_Pitch2.54mm, F.Cu at (98.5, 173.7)
- added J18: Conn_Coaxial, raisin:RFCONNECTOR, F.Cu at (83.8, 136.4)
- added J19: S-metr, Pin_Headers:Pin_Header_Straight_1x02_Pitch2.54mm, F.Cu at (58.0, 78.3)
- added J20: AGC_OFF, Pin_Headers:Pin_Header_Straight_1x02_Pitch2.54mm, F.Cu at (58.0, 86.5)
- added J21: TX_SYNT, Pin_Headers:Pin_Header_Straight_1x02_Pitch2.54mm, F.Cu at (56.1, 51.0)
- added K1: RS-12, raisin:RS-12, F.Cu at (132.8, 64.6)
- added K2: RS-12, raisin:RS-12, F.Cu at (130.7, 116.5)
- added L12: 22uH, Resistors_ThroughHole:R_Axial_DIN0207_L6.3mm_D2.5mm_P10.16mm_Horizontal, F.Cu at (100.7, 71.5)
- added L13: L_Small, raisin:Choke_Toroid_6,5x13mm_Vertical, F.Cu at (135.3, 142.3)
- added L14: 22uH, Resistors_ThroughHole:R_Axial_DIN0207_L6.3mm_D2.5mm_P10.16mm_Horizontal, F.Cu at (104.6, 127.6)
- added L15: 47uH, Resistors_ThroughHole:R_Axial_DIN0204_L3.6mm_D1.6mm_P7.62mm_Horizontal, F.Cu at (87.4, 134.3)
- added L16: L_Small, raisin:Choke_Toroid_6,5x13mm_Vertical, F.Cu at (72.5, 126.3)
- added Q12: MMBT2222, TO_SOT_Packages_SMD:SOT-23, B.Cu at (137.3, 108.9)
- added Q13: MMBFJ310LT1G, TO_SOT_Packages_SMD:SOT-23, B.Cu at (90.7, 37.5)
- added Q14: MMBFJ310LT1G, TO_SOT_Packages_SMD:SOT-23, B.Cu at (95.3, 43.9)
- added Q16: MMBFJ310LT1G, TO_SOT_Packages_SMD:SOT-23, B.Cu at (97.7, 74.0)
- added Q17: MMBFJ310LT1G, TO_SOT_Packages_SMD:SOT-23, B.Cu at (92.5, 67.0)
- added Q18: MMBFJ310LT1G, TO_SOT_Packages_SMD:SOT-23, B.Cu at (113.6, 124.2)
- added Q19: MMBT2222LT1G, TO_SOT_Packages_SMD:SOT-23, B.Cu at (120.5, 139.8)
- added Q20: BSS138, TO_SOT_Packages_SMD:SOT-23, B.Cu at (128.6, 155.0)
- added R22: 220, raisin:R_1206_0603, B.Cu at (89.2, 43.9)
- added R48: 1.5k*, raisin:R_1206_0603, B.Cu at (94.7, 61.9)
- added R49: 1.5k*, raisin:R_1206_0603, B.Cu at (92.0, 74.0)
- added R50: 30, raisin:R_1206_0603, B.Cu at (99.4, 54.8)
- added R51: 1k, raisin:R_1206_0603, B.Cu at (105.8, 98.2)
- added R52: 100R, raisin:R_1206_0603, B.Cu at (119.1, 143.2)
- added R53: 100k, raisin:R_1206_0603, B.Cu at (117.0, 139.8)
- added R54: 200k, raisin:R_1206_0603, B.Cu at (114.2, 139.8)
- added R55: 30, raisin:R_1206_0603, B.Cu at (116.5, 118.9)
- added R56: 750*, raisin:R_1206_0603, B.Cu at (125.2, 136.6)
- added R57: 10k, raisin:R_1206_0603, B.Cu at (108.2, 125.2)
- added R58: 1k, raisin:R_1206_0603, B.Cu at (123.6, 157.0)
- added R59: 15k, raisin:R_1206_0603, B.Cu at (123.7, 154.7)
- added R60: 1k, raisin:R_1206_0603, B.Cu at (80.6, 126.3)
- added R61: 1k, raisin:R_1206_0603, B.Cu at (83.7, 129.8)
- added RV2: 1M, Potentiometers:Potentiometer_Trimmer_Piher_PT-6v_Horizontal, F.Cu at (91.0, 88.1)
- added RV4: 33k, Potentiometers:Potentiometer_Trimmer_Piher_PT-6v_Horizontal, F.Cu at (72.2, 105.2)
- added RV6: 1k, Potentiometers:Potentiometer_Trimmer_Piher_PT-6v_Horizontal, F.Cu at (82.2, 104.9)
- added T5: Transformer, raisin:TF14, F.Cu at (91.9, 49.9)
- added T6: Transformer, raisin:TF14, F.Cu at (88.5, 79.4)
- added T7: Transformer, raisin:TF14, F.Cu at (120.9, 51.8)
- added T8: Transformer, raisin:TF14, F.Cu at (125.0, 118.8)
- added U9: L78L06_TO92, TO_SOT_Packages_THT:TO-92_Inline_Wide, F.Cu at (60.7, 125.4)
- added Y14: Crystal_GND23_Small, raisin:Crystal_HC49-U_Vertical, F.Cu at (82.2, 57.0)
- added Y15: Crystal_GND23_Small, raisin:Crystal_HC49-U_Vertical_4GND, F.Cu at (130.3, 89.3)
- added Y16: Crystal_GND23_Small, raisin:Crystal_HC49-U_Vertical_3GND, F.Cu at (119.0, 89.3)
- added Y17: Crystal_GND23_Small, raisin:Crystal_HC49-U_Vertical, F.Cu at (77.3, 62.1)
- added Y18: Crystal_GND23_Small, raisin:Crystal_HC49-U_Vertical_3GND, F.Cu at (125.4, 94.4)
- added Y19: Crystal_GND23_Small, raisin:Crystal_HC49-U_Vertical_4GND, F.Cu at (114.2, 94.3)
- added Y20: Crystal_GND23_Small, raisin:Crystal_HC49-U_Vertical, F.Cu at (82.2, 67.2)
- added Y21: Crystal_GND23_Small, raisin:Crystal_HC49-U_Vertical_4GND, F.Cu at (130.3, 104.6)
- added Y22: Crystal_GND23_Small, raisin:Crystal_HC49-U_Vertical_4GND, F.Cu at (130.3, 99.5)
- added Y23: Crystal_GND23_Small, raisin:Crystal_HC49-U_Vertical_3GND, F.Cu at (119.1, 104.6)
- added Y24: Crystal_GND23_Small, raisin:Crystal_HC49-U_Vertical_3GND, F.Cu at (119.0, 99.5)
- added Y25: Crystal_GND23_Small, raisin:Crystal_HC49-U_Vertical, F.Cu at (77.3, 72.3)
- added Y26: Crystal_GND23_Small, raisin:Crystal_HC49-U_Vertical, F.Cu at (77.3, 77.4)
- added Y27: Crystal_GND23_Small, raisin:Crystal_HC49-U_Vertical, F.Cu at (123.1, 134.0)
- added Y28: Crystal_GND23_Small, raisin:Crystal_HC49-U_Vertical, F.Cu at (83.5, 117.9)
- C1, C15, C25, C35, C5, C6, C85, C88, C9: footprint Capacitors_SMD:C_0603_HandSoldering -> raisin:C_1206_0603; moved to B.Cu
- C10: value 10uF -> 100nF; footprint Capacitors_ThroughHole:CP_Radial_D4.0mm_P2.00mm -> raisin:C_1206_0603
- C11: value 10nF -> 100nF; moved to B.Cu
- C12, C74: value 10nF -> 100nF; footprint Capacitors_SMD:C_0603_HandSoldering -> raisin:C_1206_0603; moved to B.Cu
- C13, C17, C2, D17, D3, D4, D5, D6, Q11, Q3, Q5, Q8: moved to B.Cu
- C14: value 10nF -> 33uF; footprint Capacitors_SMD:C_0603_HandSoldering -> Capacitors_ThroughHole:CP_Radial_D6.3mm_P2.50mm
- C16: value 10nF -> 1uF; footprint Capacitors_SMD:C_0603_HandSoldering -> Capacitors_ThroughHole:CP_Radial_D4.0mm_P2.00mm
- C19: value 100nF -> 1uF; footprint Capacitors_SMD:C_0603_HandSoldering -> raisin:C_1206_0603; moved to B.Cu
- C20, C22: value 220nF -> 1uF; moved to B.Cu
- C21: value 220nF -> 100nF; footprint raisin:C_1206_0603 -> Capacitors_SMD:C_0603_HandSoldering; moved to B.Cu
- C23: value 220nF -> 4n7; moved to B.Cu
- C24: value 10nF -> 47n; footprint Capacitors_SMD:C_0603_HandSoldering -> raisin:C_1206_0603; moved to B.Cu
- C26: value 220nF -> 10uF; footprint raisin:C_1206_0603 -> Capacitors_ThroughHole:CP_Radial_D4.0mm_P2.00mm
- C27, C72, C86, C87: value 100nF -> 10nF; moved to B.Cu
- C28: value 220nF -> 100nF; moved to B.Cu
- C29: value 33uF -> 100pF*; footprint Capacitors_ThroughHole:CP_Radial_D6.3mm_P2.50mm -> raisin:C_1206_0603
- C30: value 220nF -> 100pF*; moved to B.Cu
- C33: value 100nF -> 10uF; footprint Capacitors_SMD:C_0603_HandSoldering -> Capacitors_ThroughHole:CP_Radial_D4.0mm_P2.00mm
- C34: value 1uF -> 330uF; footprint Capacitors_ThroughHole:CP_Radial_D4.0mm_P2.00mm -> Capacitors_ThroughHole:CP_Radial_D10.0mm_P5.00mm; moved to F.Cu
- C36, C38, C47, C49, C60: value 100nF -> 100pF*; footprint Capacitors_SMD:C_0603_HandSoldering -> raisin:C_1206_0603; moved to B.Cu
- C37: value 75* -> 220uF; footprint raisin:C_1206_0603 -> Capacitors_ThroughHole:CP_Radial_D6.3mm_P2.50mm
- C39: value 10nF -> 100pF*; footprint Capacitors_SMD:C_0603_HandSoldering -> raisin:C_1206_0603; moved to B.Cu
- C41: value 10nF -> 100pF*; moved to B.Cu
- C44: value 270 -> 100nF; moved to B.Cu
- C45, C64: value 27 -> 100pF*; moved to B.Cu
- C46, C65: value 33 -> 100pF*; moved to B.Cu
- C48, C66: value 680 -> 100pF*; moved to B.Cu
- C52: value 10uF -> 100pF*; footprint Capacitors_ThroughHole:CP_Radial_D5.0mm_P2.50mm -> raisin:C_1206_0603
- C63: value 22 -> 100pF*; moved to B.Cu
- C67: value 22 -> 100nF; moved to B.Cu
- C68: value 27 -> 100nF; moved to B.Cu
- C69: value 33 -> 10nF; footprint raisin:C_1206_0603 -> Capacitors_SMD:C_0603_HandSoldering; moved to B.Cu
- C73: value 33uF -> 10nF; footprint Capacitors_ThroughHole:CP_Radial_D6.3mm_P2.50mm -> Capacitors_SMD:C_0603_HandSoldering
- C76: value 330uF -> 100nF; footprint Capacitors_ThroughHole:CP_Radial_D8.0mm_P5.00mm -> raisin:C_1206_0603
- C77: value 100uF -> 100nF; footprint Capacitors_ThroughHole:CP_Radial_D6.3mm_P2.50mm -> raisin:C_1206_0603
- C79, C83, C84: value 100pF -> 100nF; moved to B.Cu
- C80, C82: value 100pF -> 22uF; footprint raisin:C_1206_0603 -> Capacitors_ThroughHole:CP_Radial_D6.3mm_P2.50mm
- D1, D2: value LL4148 -> BAV99; footprint Diodes_SMD:D_MiniMELF -> TO_SOT_Packages_SMD:SOT-23; moved to B.Cu
- D10: value LL4148 -> D; moved to B.Cu
- D11: value BB132 -> D; footprint Diodes_SMD:D_SOD-323_HandSoldering -> Diodes_SMD:D_MiniMELF; moved to B.Cu
- D12, D13, D15: value BB132 -> LL4148; footprint Diodes_SMD:D_SOD-323_HandSoldering -> Diodes_SMD:D_MiniMELF; moved to B.Cu
- D16: value BB132 -> SS14; footprint Diodes_SMD:D_SOD-323_HandSoldering -> Diodes_SMD:D_SMA-SMB_Universal_Handsoldering; moved to B.Cu
- D7: value BAV99 -> LL4148; footprint TO_SOT_Packages_SMD:SOT-23 -> Diodes_SMD:D_MiniMELF; moved to B.Cu
- D9: value BB132 -> BAV99; footprint Diodes_SMD:D_SOD-323_HandSoldering -> TO_SOT_Packages_SMD:SOT-23; moved to B.Cu
- J1: value CW_KEY -> CW; moved to F.Cu
- J10: value Encoder -> ATT; footprint raisin:Encoder_DY-40 -> Pin_Headers:Pin_Header_Straight_1x02_Pitch2.54mm; moved to F.Cu
- J11: value i2c -> Speaker; footprint raisin:SSD1306 -> Pin_Headers:Pin_Header_Straight_1x02_Pitch2.54mm; moved to F.Cu
- J12: value Barrel_Jack -> POWER; footprint Connect:BARREL_JACK -> Connectors_Molex:Molex_KK-41791-02_02x3.96mm_Straight; moved to F.Cu
- J13: value PA -> BPF; footprint Connectors_Molex:Molex_KK-41791-02_02x3.96mm_Straight -> Pin_Headers:Pin_Header_Straight_1x02_Pitch2.54mm; moved to F.Cu
- J14: value Conn_01x02 -> AMP; moved to F.Cu
- J15, T2, Y11, Y7, Y8: moved to F.Cu
- J2: value Line OUT -> Conn_Coaxial; footprint raisin:audio_jack_3_5mm_PJ307 -> raisin:RFCONNECTOR; moved to F.Cu
- J3: value MIC -> Conn_Coaxial; footprint raisin:audio_jack_3_5mm_PJ307 -> raisin:RFCONNECTOR; moved to F.Cu
- J4: value ANT_PA -> Line OUT; footprint raisin:RFCONNECTOR -> raisin:audio_jack_3_5mm_PJ307; moved to F.Cu
- J9: value PTT -> Key; moved to F.Cu
- L11: value 8.5uH -> 47uH; footprint raisin:Choke_Toroid_6,5x13mm_Vertical -> Resistors_ThroughHole:R_Axial_DIN0204_L3.6mm_D1.6mm_P7.62mm_Horizontal; moved to F.Cu
- L3, L4: value 22uH -> L; footprint Resistors_ThroughHole:R_Axial_DIN0204_L3.6mm_D1.6mm_P7.62mm_Horizontal -> Choke_Toroid_ThroughHole:Choke_Toroid_6,5x13mm_Vertical; moved to F.Cu
- L6: value 47uH -> 22uH; footprint Resistors_ThroughHole:R_Axial_DIN0204_L3.6mm_D1.6mm_P7.62mm_Horizontal -> Resistors_ThroughHole:R_Axial_DIN0207_L6.3mm_D2.5mm_P10.16mm_Horizontal; moved to F.Cu
- L8: value 8.5uH -> 22uH; footprint raisin:Choke_Toroid_6,5x13mm_Vertical -> Resistors_ThroughHole:R_Axial_DIN0207_L6.3mm_D2.5mm_P10.16mm_Horizontal; moved to F.Cu
- Q1, Q2: value MMBFJ310LT1G -> Si2301-TP; moved to B.Cu
- Q4: value Si2301-TP -> MMBT3906; moved to B.Cu
- Q7: value MMBFJ310LT1G -> 2N7002; moved to B.Cu
- R10: value 10k -> 4.7k; moved to B.Cu
- R11: value 2.7k -> 4.7k; moved to B.Cu
- R12: value 2.7k -> 4.7k; footprint raisin:R_1206_0603 -> Resistors_SMD:R_0603_HandSoldering; moved to B.Cu
- R13: value 10k -> 150k*; footprint Resistors_SMD:R_0603_HandSoldering -> raisin:R_1206_0603; moved to B.Cu
- R14: value 30 -> 100; moved to B.Cu
- R15: value 4.7k -> 100; footprint Resistors_SMD:R_0603_HandSoldering -> raisin:R_1206_0603; moved to B.Cu
- R16: value 4.7k -> 150k*; footprint Resistors_SMD:R_0603_HandSoldering -> raisin:R_1206_0603; moved to B.Cu
- R17: value 100 -> 15k; moved to B.Cu
- R18: value 100 -> 1k; footprint raisin:R_1206_0603 -> Resistors_ThroughHole:R_Axial_DIN0204_L3.6mm_D1.6mm_P7.62mm_Horizontal
- R19: value 3,3k -> 15k; moved to B.Cu
- R2, R7, R8: value 300k -> 2.7k; moved to B.Cu
- R20: value 3,3k -> 2k; moved to B.Cu
- R23: value 150k* -> 12k; moved to B.Cu
- R24: value 30 -> 2.2k; moved to B.Cu
- R25: value 15 -> 30; moved to B.Cu
- R26: value 10k -> 2.2k; footprint Resistors_SMD:R_0603_HandSoldering -> raisin:R_1206_0603; moved to B.Cu
- R28: value 1k -> 220; footprint Resistors_SMD:R_0603_HandSoldering -> raisin:R_1206_0603; moved to B.Cu
- R3: value 10k -> 1M; footprint Resistors_SMD:R_0603_HandSoldering -> Resistors_SMD:R_1206_HandSoldering
- R32: value 1k -> 0*; footprint Resistors_SMD:R_0603_HandSoldering -> raisin:R_1206_0603; moved to B.Cu
- R36: value 300k -> 30; moved to B.Cu
- R38: value 300k -> 1M; footprint raisin:R_1206_0603 -> Resistors_SMD:R_1206_HandSoldering; moved to B.Cu
- R42: value 10k -> 3,3k; footprint Resistors_SMD:R_0603_HandSoldering -> raisin:R_1206_0603; moved to B.Cu
- R44: value 470k -> 3,3k; moved to B.Cu
- R45: value 470k -> 4.7k; moved to B.Cu
- R47: value 0* -> 30; moved to B.Cu
- R9: value 30 -> 2.7k; moved to B.Cu
- T1: footprint raisin:TF12 -> raisin:TF_2; moved to F.Cu
- U1: value ATMEGA328P-AU -> NE5532; footprint Housings_QFP:TQFP-32_7x7mm_Pitch0.8mm -> Housings_SOIC:SOIC-8_3.9x4.9mm_Pitch1.27mm; moved to B.Cu
- U2: value Si5351 -> TDA7052A; footprint Housings_SSOP:MSOP-10_3x3mm_Pitch0.5mm -> Housings_DIP:DIP-8_W7.62mm
- U3: value NE5532 -> NC7WZ04; footprint Housings_SOIC:SOIC-8_3.9x4.9mm_Pitch1.27mm -> TO_SOT_Packages_SMD:SOT-363_SC-70-6_Handsoldering; moved to B.Cu
- U5: value LD1117S33TR_SOT223 -> L78L05_TO92; footprint TO_SOT_Packages_SMD:SOT-223-3_TabPin2 -> TO_SOT_Packages_THT:TO-92_Inline_Wide
- U6: value L78L05_TO92 -> FSA3157L6X; footprint TO_SOT_Packages_THT:TO-92_Molded_Wide -> TO_SOT_Packages_SMD:SOT-23-6_Handsoldering
- U7: value FSA3157L6X -> SA612A; footprint TO_SOT_Packages_SMD:SOT-363_SC-70-6_Handsoldering -> raisin:DIP-8_SOIC-8_W7.62mm
- Y10, Y12, Y4: footprint raisin:Crystal_HC49-U_Vertical -> raisin:Crystal_HC49-U_Vertical_3GND; moved to F.Cu
- Y13, Y5, Y6, Y9: footprint raisin:Crystal_HC49-U_Vertical -> raisin:Crystal_HC49-U_Vertical_4GND; moved to F.Cu
- Y2: value 27Mhz -> Crystal_GND23_Small; footprint Crystals:Crystal_SMD_HC49-SD -> raisin:Crystal_HC49-U_Vertical_3GND
- moved J10 124.1 mm to (56.1, 35.8), turned to 0 degrees
- moved J4 112.4 mm to (101.0, 160.0), turned to 180 degrees
- moved R32 110.4 mm to (60.8, 117.0), turned to 90 degrees
- moved J8 105.6 mm to (57.5, 23.0)
- moved R26 100.5 mm to (60.3, 48.8), turned to 270 degrees
- moved C77 99.8 mm to (135.5, 37.0), turned to 90 degrees
- moved R12 99.1 mm to (63.4, 66.5), turned to 180 degrees
- moved C1 96.1 mm to (69.2, 54.9), turned to 180 degrees
- moved J11 95.4 mm to (58.0, 93.5), turned to 0 degrees
- moved C38 94.1 mm to (79.8, 49.4)
- moved L6 93.8 mm to (106.1, 34.4), turned to 180 degrees
- moved Q7 90.7 mm to (65.0, 50.0)
- moved C34 90.2 mm to (61.0, 37.9), turned to 0 degrees
- moved C44 89.6 mm to (140.5, 110.3), turned to 270 degrees
- moved D16 89.1 mm to (67.5, 27.1)
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Connections:
- C1 pad 1: GNDD -> +12V
- C1 pad 2: +3V3 -> Net-(C1-Pad2)
- C11 pad 1: Net-(C11-Pad1) -> TX
- C11 pad 2: Net-(C11-Pad2) -> GND
- C12 pad 1: Net-(C12-Pad1) -> CW_TONE
- C12 pad 2: Net-(C12-Pad2) -> GND
- C13 pad 1: +12V -> RX
- C13 pad 2: Net-(C13-Pad2) -> GND
- C14 pad 2: Net-(C14-Pad2) -> GND
- C15 pad 1: Net-(C15-Pad1) -> Net-(C14-Pad1)
- C15 pad 2: Net-(C15-Pad2) -> GND
- C16 pad 2: Net-(C16-Pad2) -> GND
- C17 pad 1: TX -> Net-(C17-Pad1)
- C17 pad 2: GND -> Net-(C17-Pad2)
- C19 pad 1: RX -> Net-(C17-Pad1)
- C19 pad 2: GND -> Net-(C19-Pad2)
- C2 pad 1: GNDD -> +12V
- C20 pad 2: Net-(C20-Pad2) -> GND
- C23 pad 2: Net-(C23-Pad2) -> GND
- C24 pad 2: VFO -> Net-(C17-Pad1)
- C27 pad 1: Net-(C27-Pad1) -> AUDIO
- C28 pad 2: Net-(C28-Pad2) -> GND
- C29 pad 1: Net-(C25-Pad1) -> Net-(C29-Pad1)
- C30 pad 2: Net-(C30-Pad2) -> GND
- C33 pad 1: Net-(C32-Pad1) -> Net-(C100-Pad1)
- C34 pad 1: Net-(C34-Pad1) -> +12V
- C35 pad 2: Net-(C35-Pad2) -> GND
- C36 pad 1: +12V -> Net-(C36-Pad1)
- C37 pad 1: Net-(C37-Pad1) -> Net-(C35-Pad1)
- C37 pad 2: Net-(C37-Pad2) -> GND
- C39 pad 2: VFO -> GND
- C41 pad 2: Net-(C41-Pad2) -> GND
- C44 pad 1: Net-(C41-Pad2) -> Net-(C44-Pad1)
- C45 pad 2: Net-(C45-Pad2) -> GND
- C46 pad 1: Net-(C45-Pad1) -> Net-(C46-Pad1)
- C46 pad 2: Net-(C45-Pad2) -> GND
- C48 pad 1: Net-(C45-Pad2) -> Net-(C48-Pad1)
- C5 pad 2: GND -> Net-(C5-Pad2)
- C52 pad 1: Net-(C47-Pad1) -> Net-(C52-Pad1)
- C6 pad 1: GND -> VCC
- C6 pad 2: TX -> GND
- C63 pad 1: Net-(C45-Pad2) -> Net-(C63-Pad1)
- C64 pad 2: Net-(C64-Pad2) -> GND
- C65 pad 1: Net-(C64-Pad1) -> Net-(C65-Pad1)
- C65 pad 2: Net-(C64-Pad2) -> GND
- C66 pad 1: Net-(C64-Pad2) -> Net-(C66-Pad1)
- C67 pad 1: Net-(C64-Pad2) -> GND
- C67 pad 2: GND -> Net-(C28-Pad1)
- C68 pad 1: Net-(C68-Pad1) -> TX
- C68 pad 2: Net-(C12-Pad1) -> GND
- C69 pad 1: Net-(C68-Pad1) -> Net-(C69-Pad1)
- C69 pad 2: Net-(C12-Pad1) -> Net-(C69-Pad2)
- C72 pad 2: GND -> Net-(C72-Pad2)
- C73 pad 1: Net-(C72-Pad1) -> Net-(C73-Pad1)
- C73 pad 2: GND -> Net-(C73-Pad2)
- C76 pad 1: +12V -> RX
- C77 pad 1: +3V3 -> Net-(C77-Pad1)
- C77 pad 2: GNDD -> GND
- C79 pad 1: Net-(C21-Pad2) -> Net-(C79-Pad1)
- C80 pad 1: Net-(C22-Pad2) -> Net-(C77-Pad1)
- C82 pad 1: Net-(C26-Pad2) -> Net-(C79-Pad1)
- C83 pad 1: Net-(C28-Pad2) -> TX
- C84 pad 1: Net-(C30-Pad2) -> Net-(C84-Pad1)
- C85 pad 1: +12V -> Net-(C85-Pad1)
- C85 pad 2: GND -> Net-(C85-Pad2)
- C86 pad 1: TX -> Net-(C86-Pad1)
- C86 pad 2: GND -> Net-(C86-Pad2)
- C87 pad 1: TX -> Net-(C87-Pad1)
- C87 pad 2: GND -> Net-(C87-Pad2)
- C88 pad 1: RX -> Net-(C88-Pad1)
- C88 pad 2: GND -> Net-(C88-Pad2)
- C9 pad 1: Net-(C10-Pad1) -> Net-(C9-Pad1)
- D1 pad 1: Net-(C11-Pad2) -> TX
- D1 pad 2: TX -> Net-(C84-Pad1)
- D10 pad 1: Net-(C49-Pad1) -> +12V
- D10 pad 2: Net-(C50-Pad1) -> Net-(C28-Pad1)
- D11 pad 1: Net-(C21-Pad2) -> +12V
- D11 pad 2: GND -> Net-(C28-Pad1)
- D12 pad 1: Net-(C22-Pad2) -> Net-(C69-Pad2)
- D12 pad 2: GND -> TX
- D13 pad 1: Net-(C23-Pad2) -> Net-(C72-Pad1)
- D13 pad 2: GND -> RX
- D15 pad 1: Net-(C28-Pad2) -> Net-(C87-Pad1)
- D15 pad 2: GND -> RX
- D16 pad 1: Net-(C30-Pad2) -> +12V
- D16 pad 2: GND -> Net-(D16-Pad2)
- D17 pad 1: Net-(C74-Pad2) -> Net-(C103-Pad1)
- D17 pad 2: Net-(C75-Pad1) -> RX
- D2 pad 1: PTT -> Net-(C86-Pad2)
- D2 pad 2: Net-(D2-Pad2) -> Net-(C86-Pad2)
- D3 pad 1: Net-(C14-Pad1) -> Net-(D3-Pad1)
- D3 pad 2: RX -> Net-(D3-Pad2)
- D4 pad 1: Net-(C31-Pad1) -> TX
- D4 pad 2: Net-(C37-Pad1) -> CW_TONE
- D5 pad 1: Net-(C37-Pad1) -> Net-(C14-Pad1)
- D5 pad 2: TX -> Net-(C17-Pad2)
- D6 pad 1: Net-(C32-Pad1) -> Net-(C96-Pad1)
- D6 pad 2: Net-(C42-Pad2) -> Net-(C106-Pad1)
- D7 pad 1: GND -> Net-(C106-Pad1)
- D7 pad 2: Net-(C34-Pad1) -> TX
- D9 pad 1: Net-(C20-Pad2) -> GND
- D9 pad 2: GND -> Net-(C16-Pad1)
- J1 pad 1: Net-(J1-Pad1) -> CW
- J1 pad 2: Net-(J1-Pad2) -> GND
- J10 pad 1: GNDD -> +12V
- J10 pad 2: +3V3 -> GND
- J11 pad 1: GNDD -> Net-(J11-Pad1)
- J11 pad 2: +3V3 -> Net-(J11-Pad2)
- J12 pad 1: +12V -> Net-(D16-Pad2)
- J14 pad 1: Net-(J14-Pad1) -> Net-(C20-Pad1)
- J14 pad 2: Net-(J14-Pad2) -> GND
- J2 pad 1: Net-(C91-Pad2) -> VFO
- J2 pad 2: Net-(C91-Pad2) -> GND
- J3 pad 1: Net-(C57-Pad1) -> BPF
- J3 pad 2: Net-(C57-Pad1) -> GND
- J4 pad 1: Net-(C41-Pad1) -> Net-(C22-Pad2)
- J4 pad 2: GND -> Net-(C22-Pad2)
- J9 pad 1: Net-(J9-Pad1) -> Net-(D3-Pad1)
- J9 pad 2: Net-(J9-Pad2) -> Net-(D3-Pad1)
- J9 pad 3: GNDD -> GND
- J9 pad 4: Net-(J9-Pad1) -> Net-(D3-Pad1)
- J9 pad 5: Net-(J9-Pad2) -> Net-(D3-Pad1)
- L11 pad 1: Net-(C64-Pad2) -> Net-(C77-Pad1)
- L11 pad 2: Net-(C68-Pad1) -> VCC
- L3 pad 1: GND -> Net-(C29-Pad1)
- L4 pad 1: Net-(C11-Pad2) -> Net-(L4-Pad1)
- L4 pad 2: Net-(C14-Pad1) -> Net-(C66-Pad1)
- L6 pad 1: +3V3 -> GND
- L6 pad 2: Net-(C47-Pad1) -> Net-(L6-Pad2)
- L8 pad 1: Net-(C41-Pad2) -> Net-(C69-Pad2)
- L8 pad 2: Net-(C45-Pad1) -> Net-(C72-Pad1)
- Q1 pad 1: Net-(C11-Pad2) -> Net-(C1-Pad2)
- Q1 pad 2: Net-(C16-Pad1) -> +12V
- Q1 pad 3: Net-(C14-Pad2) -> TX
- Q11 pad 1: AGC_OFF -> TX
- Q11 pad 3: Net-(C32-Pad1) -> Net-(C20-Pad1)
- Q2 pad 1: Net-(C14-Pad1) -> Net-(C2-Pad2)
- Q2 pad 2: Net-(C15-Pad2) -> +12V
- Q2 pad 3: Net-(C11-Pad1) -> CW_TONE
- Q3 pad 1: Net-(C13-Pad2) -> TX
- Q3 pad 3: TX -> RX
- Q4 pad 1: TX -> Net-(C16-Pad1)
- Q4 pad 2: +12V -> Net-(C14-Pad1)
- Q4 pad 3: RX -> GND
- Q5 pad 1: Net-(C32-Pad1) -> Net-(C9-Pad1)
- Q5 pad 3: AGC -> Net-(C14-Pad1)
- Q7 pad 1: Net-(Q7-Pad1) -> Net-(C10-Pad1)
- Q7 pad 2: Net-(C35-Pad1) -> GND
- Q7 pad 3: Net-(C40-Pad2) -> Net-(Q7-Pad3)
- Q8 pad 1: Net-(Q8-Pad1) -> Net-(C14-Pad1)
- Q8 pad 3: Net-(C74-Pad2) -> AGC
- R10 pad 1: GND -> TX
- R10 pad 2: Net-(C11-Pad1) -> GND
- R11 pad 1: +12V -> CW_TONE
- R11 pad 2: Net-(C13-Pad2) -> GND
- R12 pad 1: Net-(C13-Pad2) -> RX
- R12 pad 2: Net-(D2-Pad2) -> GND
- R13 pad 1: Net-(C14-Pad2) -> Net-(C16-Pad1)
- R14 pad 1: Net-(C15-Pad1) -> Net-(C22-Pad1)
- R14 pad 2: Net-(C15-Pad2) -> Net-(C17-Pad1)
- R15 pad 1: TX -> Net-(C25-Pad1)
- R15 pad 2: GND -> RX
- R16 pad 1: RX -> Net-(C20-Pad1)
- R17 pad 1: VFO -> Net-(C24-Pad1)
- R17 pad 2: GND -> Net-(C23-Pad1)
- R18 pad 1: Net-(C25-Pad1) -> Net-(R18-Pad1)
- R19 pad 1: Net-(C27-Pad1) -> Net-(R18-Pad1)
- R19 pad 2: Net-(C25-Pad1) -> Net-(C26-Pad1)
- R2 pad 1: Net-(C20-Pad2) -> +12V
- R2 pad 2: Net-(C60-Pad1) -> Net-(C1-Pad2)
- R20 pad 1: Net-(C25-Pad1) -> Net-(C44-Pad1)
- R20 pad 2: GND -> CW
- R23 pad 1: Net-(C34-Pad1) -> S-metr
- R23 pad 2: GND -> Net-(J19-Pad1)
- R24 pad 1: Net-(C35-Pad1) -> Net-(C9-Pad1)
- R24 pad 2: Net-(C35-Pad2) -> AGC_OFF
- R25 pad 1: Net-(C37-Pad1) -> Net-(L6-Pad2)
- R25 pad 2: Net-(Q7-Pad1) -> Net-(C73-Pad1)
- R26 pad 1: Net-(C40-Pad2) -> Net-(C10-Pad1)
- R26 pad 2: GND -> TX_SYNT
- R28 pad 1: AGC -> Net-(C72-Pad2)
- R28 pad 2: Net-(C49-Pad1) -> GND
- R3 pad 1: +3V3 -> VFO
- R3 pad 2: Net-(CON1-Pad5) -> Net-(C5-Pad2)
- R32 pad 1: Net-(C57-Pad1) -> +12V
- R32 pad 2: Net-(C55-Pad1) -> Net-(C35-Pad1)
- R36 pad 1: Net-(C26-Pad2) -> Net-(C74-Pad2)
- R36 pad 2: Net-(C60-Pad1) -> Net-(C74-Pad1)
- R38 pad 1: Net-(C30-Pad2) -> Net-(C5-Pad1)
- R38 pad 2: Net-(C60-Pad1) -> Net-(R38-Pad2)
- R42 pad 1: Net-(Q8-Pad1) -> VCC
- R42 pad 2: KEY -> Net-(C79-Pad1)
- R44 pad 1: Net-(C32-Pad1) -> Net-(C79-Pad1)
- R44 pad 2: S -> GND
- R45 pad 1: S -> Net-(C84-Pad1)
- R45 pad 2: GNDD -> AGC
- R47 pad 1: Net-(C38-Pad1) -> Net-(C85-Pad2)
- R47 pad 2: Net-(C60-Pad1) -> Net-(C85-Pad1)
- R7 pad 1: Net-(C21-Pad2) -> Net-(C1-Pad2)
- R7 pad 2: Net-(C60-Pad1) -> Net-(Q7-Pad3)
- R8 pad 1: Net-(C22-Pad2) -> +12V
- R8 pad 2: Net-(C60-Pad1) -> Net-(C2-Pad2)
- R9 pad 1: Net-(L3-Pad2) -> Net-(C2-Pad2)
- R9 pad 2: Net-(C16-Pad1) -> Net-(D3-Pad2)
- T1 pad 1: GND -> BPF
- T1 pad 2: Net-(C12-Pad2) -> GND
- T2 pad 1: Net-(T1-Pad3) -> Net-(T1-Pad4)
- T2 pad 2: Net-(C16-Pad2) -> Net-(C73-Pad2)
- T2 pad 3: Net-(C16-Pad2) -> Net-(C73-Pad2)
- T2 pad 4: Net-(T1-Pad4) -> Net-(T1-Pad3)
- U1 pad 1: Net-(C94-Pad1) -> Net-(C17-Pad1)
- U1 pad 2: (no net) -> Net-(C17-Pad1)
- U1 pad 3: GNDD -> Net-(C23-Pad1)
- U1 pad 4: +3V3 -> GND
- U1 pad 5: GNDD -> AUDIO
- U1 pad 6: +3V3 -> Net-(C26-Pad1)
- U1 pad 7: Net-(C3-Pad1) -> Net-(R18-Pad1)
- U1 pad 8: Net-(C4-Pad1) -> Net-(C25-Pad1)
- U2 pad 1: Net-(C47-Pad1) -> Net-(C35-Pad1)
- U2 pad 2: Net-(U2-Pad2) -> Net-(C21-Pad1)
- U2 pad 3: Net-(U2-Pad3) -> GND
- U2 pad 4: SCL -> Net-(C20-Pad1)
- U2 pad 5: SDA -> Net-(J11-Pad1)
- U2 pad 6: Net-(C74-Pad1) -> GND
- U2 pad 7: Net-(C47-Pad1) -> (no net)
- U2 pad 8: GND -> Net-(J11-Pad2)
- U3 pad 1: Net-(R31-Pad1) -> Net-(C5-Pad1)
- U3 pad 2: Net-(C58-Pad1) -> GND
- U3 pad 3: Net-(C59-Pad1) -> VFO
- U3 pad 4: GND -> Net-(C5-Pad2)
- U3 pad 5: Net-(C51-Pad1) -> VCC
- U3 pad 6: Net-(C42-Pad1) -> Net-(R38-Pad2)
- U5 pad 1: GNDD -> Net-(C77-Pad1)
- U5 pad 2: +3V3 -> GND
- U6 pad 1: Net-(C72-Pad1) -> Net-(T1-Pad3)
- U6 pad 3: +12V -> Net-(T1-Pad4)
- U7 pad 1: Net-(T1-Pad4) -> Net-(C108-Pad2)
- U7 pad 2: GND -> Net-(C106-Pad2)
- U7 pad 3: Net-(T1-Pad3) -> GND
- U7 pad 4: Net-(C25-Pad1) -> Net-(C107-Pad2)
- U7 pad 5: Net-(C27-Pad1) -> AUDIO
- U7 pad 6: Net-(C24-Pad1) -> Net-(C112-Pad2)
- Y10 pad 1: Net-(C26-Pad1) -> Net-(C36-Pad1)
- Y10 pad 2: Net-(C28-Pad1) -> Net-(C41-Pad1)
- Y11 pad 1: Net-(C28-Pad1) -> Net-(C38-Pad1)
- Y11 pad 2: Net-(C30-Pad1) -> Net-(C45-Pad1)
- Y12 pad 1: Net-(C30-Pad1) -> Net-(C39-Pad1)
- Y12 pad 2: FILT -> Net-(C46-Pad1)
- Y13 pad 1: Net-(C30-Pad1) -> Net-(C41-Pad1)
- Y13 pad 2: FILT -> Net-(C47-Pad1)
- Y2 pad 1: Net-(U2-Pad2) -> Net-(K1-Pad1)
- Y2 pad 2: Net-(U2-Pad3) -> Net-(C30-Pad1)
- Y4 pad 1: FIL -> Net-(K1-Pad1)
- Y4 pad 2: Net-(C20-Pad1) -> Net-(C30-Pad1)
- Y5 pad 1: FIL -> Net-(L3-Pad2)
- Y5 pad 2: Net-(C20-Pad1) -> Net-(C36-Pad1)
- Y6 pad 1: Net-(C20-Pad1) -> Net-(L3-Pad2)
- Y6 pad 2: Net-(C21-Pad1) -> Net-(C36-Pad1)
- Y7 pad 1: Net-(C21-Pad1) -> QER11
- Y7 pad 2: Net-(C22-Pad1) -> Net-(C38-Pad1)
- Y8 pad 1: Net-(C22-Pad1) -> QER11
- Y8 pad 2: Net-(C23-Pad1) -> Net-(C38-Pad1)
- Y9 pad 1: Net-(C23-Pad1) -> Net-(C30-Pad1)
- Y9 pad 2: Net-(C26-Pad1) -> Net-(C39-Pad1)
Routing:
- net GND: track 798.9 -> 39.6 mm, vias 191 -> 13
- net GNDD: track 188.0 -> 0.00 mm, vias 42 -> 0
- net +3V3: track 124.3 -> 0.00 mm, vias 1 -> 0
- net Net-(C13-Pad2): track 116.5 -> 0.00 mm, vias 2 -> 0
- net Net-(C32-Pad1): track 116.0 -> 0.00 mm, vias 2 -> 0
- net RX: track 166.4 -> 281.7 mm, vias 2 -> 4
- net SDA: track 101.3 -> 0.00 mm, vias 2 -> 0
- net SCL: track 97.6 -> 0.00 mm, vias 2 -> 0
- net Net-(C60-Pad1): track 89.4 -> 6.39 mm, vias 2 -> 0
- net Net-(C17-Pad1): track 0.00 -> 76.7 mm, vias 0 -> 2
- net Net-(C108-Pad1): track 0.00 -> 67.1 mm
- net TX: track 167.0 -> 229.4 mm, vias 2 -> 6
- net PTT: track 58.6 -> 0.00 mm
- net Net-(C28-Pad1): track 6.35 -> 59.7 mm
- net Net-(C27-Pad1): track 43.9 -> 0.00 mm, vias 1 -> 0
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- removed copper zone on B.Cu, net GNDD
- removed copper zone on F.Cu, net GNDD
Other:
- board size 95.5 x 100 mm -> 90 x 144.6 mm
- net class Default: trace_width 0.25 -> 0.3

Commit message: DX PCB
Parts:
- C11, C13: footprint Capacitors_SMD:C_0603_HandSoldering -> raisin:C_1206_0603
- R10, R12: footprint Resistors_SMD:R_0603_HandSoldering -> raisin:R_1206_0603
- moved J17 111.3 mm to (58.1, 70.0)
- moved R10 7.82 mm to (58.5, 58.0)
- moved R11 5.96 mm to (113.4, 145.1)
- moved R12 5.83 mm to (62.5, 72.3)
- moved C11 4.93 mm to (58.5, 61.9)
- moved R26 4.66 mm to (63.9, 45.8), turned to 180 degrees
- moved C10 3.78 mm to (68.9, 45.8)
- moved C73 3.68 mm to (97.2, 31.9)
- moved Q1 3.00 mm to (66.0, 60.9)
- moved Q3 3.00 mm to (65.2, 65.5)
- moved R24 3.00 mm to (62.0, 86.5)
- moved Q7 2.47 mm to (67.3, 49.0)
- moved C1 2.00 mm to (67.2, 54.9)
- moved R2 2.00 mm to (67.1, 57.5)
- moved R7 2.00 mm to (63.0, 54.4)
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Routing:
- net +12V: track 293.3 -> 404.9 mm
- net TX: track 229.4 -> 281.8 mm, vias 6 -> 4
- net GND: track 39.6 -> 59.1 mm, vias 13 -> 20
- net Net-(C5-Pad2): track 0.00 -> 6.14 mm
- net Net-(Q7-Pad3): track 2.20 -> 7.41 mm
- net Net-(C73-Pad2): track 22.4 -> 27.5 mm
- net TX_SYNT: track 5.31 -> 9.92 mm
- net Net-(C73-Pad1): track 16.5 -> 12.9 mm
- net Net-(C10-Pad1): track 8.35 -> 4.81 mm
- net Net-(C9-Pad1): track 16.7 -> 19.7 mm
- net AGC_OFF: track 0.00 -> 2.80 mm
- net RX: track 281.7 -> 283.8 mm
- net CW_TONE: track 21.3 -> 19.5 mm
- net VFO: track 14.0 -> 15.6 mm
